Commit message: add realsenseD435

File: p3at_description/urdf/robot.urdf.xacro (robot description, xacro)
@@ -14,6 +14,11 @@
   <!-- camera -->
   <xacro:include filename="$(find p3at_description)/urdf/camera_rc2016.urdf.xacro"/>
-  <xacro:camera_rc2016 parent="base_link" name="camera" topic="/camera/image_raw">
+  <xacro:camera_rc2016 parent="base_link" name="rc2016" topic="/camera/image_raw">
     <origin xyz="0.0675 0.2 0.54" rpy="0 -0 1.5707" />
   </xacro:camera_rc2016>
+  <!-- realsense d435 -->
+  <xacro:include filename="$(find realsense_gazebo_plugin)/urdf/realsense_d435.urdf.xacro"/>
+  <xacro:realsense_d435 parent="base_link">
+    <origin xyz="0.0 0 0.54" rpy="1.5707 0 1.5707" />
+  </xacro:realsense_d435>
 </robot>

Commit message: added the model of suv

File: p3at_description/urdf/robot.urdf.xacro (robot description, xacro)
@@ -17,8 +17,13 @@
     <origin xyz="0.0675 0.2 0.54" rpy="0 -0 1.5707" />
   </xacro:camera_rc2016>
-  <!-- realsense d435 -->
+  <!-- realsense d435
   <xacro:include filename="$(find realsense_gazebo_plugin)/urdf/realsense_d435.urdf.xacro"/>
   <xacro:realsense_d435 parent="base_link">
     <origin xyz="0.0 0 0.54" rpy="1.5707 0 1.5707" />
-  </xacro:realsense_d435>
+  </xacro:realsense_d435> -->
+  <!-- realsense d455 -->
+  <xacro:include filename="$(find realsense_gazebo_plugin)/urdf/realsense_d455.urdf.xacro"/>
+  <xacro:realsense_d455 parent="base_link">
+    <origin xyz="0.0 0 0.54" rpy="1.5707 0 1.5707" />
+  </xacro:realsense_d455>
 </robot>

Commit message: added depthmap processing function

File: p3at_description/urdf/robot.urdf.xacro (robot description, xacro)
@@ -1,4 +1,5 @@
 <?xml version="1.0"?>
 <robot xmlns:xacro="http://www.ros.org/wiki/xacro" name="example">
+  <xacro:arg name="camera_height" default="1.9"/>
   <xacro:arg name="gpu" default="false"/>
   <xacro:property name="gpu" value="$(arg gpu)" />
@@ -10,5 +11,5 @@
   <xacro:include filename="$(find p3at_description)/urdf/velodyne.urdf.xacro"/>
   <xacro:HDL-32E parent="base_link" name="velodyne" topic="/velodyne_points" organize_cloud="${organize_cloud}" hz="10" samples="440" gpu="${gpu}">
-    <origin xyz="0 0 0.7" rpy="0 0 0" />
+    <origin xyz="0 0 1.5" rpy="0 0 0" />
   </xacro:HDL-32E>
   <!-- camera -->
@@ -25,5 +26,5 @@
   <xacro:include filename="$(find realsense_gazebo_plugin)/urdf/realsense_d455.urdf.xacro"/>
   <xacro:realsense_d455 parent="base_link">
-    <origin xyz="0.0 0 0.54" rpy="1.5707 0 1.5707" />
+    <origin xyz="0.0 0 $(arg camera_height)" rpy="1.5707 0 1.5707" />
   </xacro:realsense_d455>
 </robot>
