Commit message: added velodyne

File: p3at_description/urdf/pioneer3at.urdf.xacro (robot description, xacro)
@@ -7,19 +7,4 @@
 <!-- Chassis -->
 	<link name="base_link">
-		<inertial>
-			<!-- default -->
-			<!-- P3AT 18.6kg plus three batteries @ 2.4kg each  minus four wheels @ 1.4 kg ea and top plate @ 0.1 kg-->
-			<mass value="21.5"/>
-			<origin xyz="-0.1 0 0.177"/>
-			<inertia ixx="0.3338" ixy="0.0"     ixz="0.0"
-				              iyy="0.4783"  iyz="0.0"
-				                            izz="0.3338"/>
-			<!-- from new3.world of p3at -->
-			<!-- <mass value="14.27"/>
-			<origin xyz="-0.1 0 0.177"/>
-			<inertia ixx="0.192883" ixy="-0.00357616"     ixz="-0.0064908"
-				              iyy="0.371329"  iyz="-0.019232"
-				                            izz="0.4098"/>		 -->
-		</inertial>
 		<visual>
 			<origin xyz="0 0 0.177" rpy="0 0 0"/>
@@ -41,4 +26,21 @@
 		<material value="Gazebo/Red"/>
 	</gazebo>
+	<link name="dummy_link">
+		<!-- Defining the inertia properties of virtual links -->
+		<inertial>
+				<!-- default -->
+				<!-- P3AT 18.6kg plus three batteries @ 2.4kg each  minus four wheels @ 1.4 kg ea and top plate @ 0.1 kg-->
+				<mass value="21.5"/>
+				<origin xyz="-0.1 0 0.177"/>
+				<inertia ixx="0.3338" ixy="0.0"     ixz="0.0"
+								iyy="0.4783"  iyz="0.0"
+												izz="0.3338"/>
+		</inertial>
+	</link>
+	<joint name="dummy_joint" type="fixed">
+		<origin rpy="0 0 0" xyz="0 0 0"/>
+		<parent link="base_link"/> <!-- Connect to the actual link -->
+		<child link="dummy_link"/>   <!-- Connect to the dummy link -->
+	</joint>
 <!-- Top -->
 	<link name="top_plate">

File: p3at_description/urdf/robot.urdf.xacro (robot description, xacro)
@@ -7,5 +7,4 @@
   <!-- pioneer3at  -->
   <xacro:include filename="$(find p3at_description)/urdf/pioneer3at.urdf.xacro"/>
-    <origin xyz="6 10 0" rpy="0 0 0" />
   <!-- velodyne -->
   <xacro:include filename="$(find p3at_description)/urdf/velodyne.urdf.xacro"/>

Commit message: final version

File: p3at_description/urdf/pioneer3at.urdf.xacro (robot description, xacro)
@@ -31,6 +31,6 @@
 				<!-- default -->
 				<!-- P3AT 18.6kg plus three batteries @ 2.4kg each  minus four wheels @ 1.4 kg ea and top plate @ 0.1 kg-->
-				<mass value="21.5"/>
-				<origin xyz="-0.1 0 0.177"/>
+				<mass value="18.6"/>
+				<origin xyz="-0.1 0 0"/>
 				<inertia ixx="0.3338" ixy="0.0"     ixz="0.0"
 								iyy="0.4783"  iyz="0.0"
@@ -339,5 +339,5 @@
   <plugin name="skid_steer_drive_controller" filename="libgazebo_ros_skid_steer_drive.so">
     <updateRate>100.0</updateRate>
-    <robotNamespace>sim_p3at</robotNamespace>
+    <robotNamespace>/</robotNamespace>
     <leftFrontJoint>p3at_front_left_wheel_joint</leftFrontJoint>
     <rightFrontJoint>p3at_front_right_wheel_joint</rightFrontJoint>
@@ -347,10 +347,7 @@
     <wheelDiameter>0.215</wheelDiameter>
     <robotBaseFrame>base_link</robotBaseFrame>
-    <MaxForce>5.0</MaxForce>
-    <torque>200</torque>
-    <commandTopic>/p3at/cmd_vel</commandTopic>
-    <odometryTopic>/p3at/odom</odometryTopic>
-    <odometryFrame>odom</odometryFrame>
-    <broadcastTF>1</broadcastTF>
+    <torque>20</torque>
+    <topicName>cmd_vel</topicName>
+    <broadcastTF>false</broadcastTF>
   </plugin>
 </gazebo>

File: p3at_description/urdf/robot.urdf.xacro (robot description, xacro)
@@ -1,5 +1,4 @@
 <?xml version="1.0"?>
 <robot xmlns:xacro="http://www.ros.org/wiki/xacro" name="example">
-  <xacro:arg name="camera_height" default="1.9"/>
   <xacro:arg name="gpu" default="false"/>
   <xacro:property name="gpu" value="$(arg gpu)" />
@@ -11,5 +10,5 @@
   <xacro:include filename="$(find p3at_description)/urdf/velodyne.urdf.xacro"/>
   <xacro:HDL-32E parent="base_link" name="velodyne" topic="/velodyne_points" organize_cloud="${organize_cloud}" hz="10" samples="440" gpu="${gpu}">
-    <origin xyz="0 0 1.5" rpy="0 0 0" />
+    <origin xyz="0 0 1.0" rpy="0 0 0" />
   </xacro:HDL-32E>
   <!-- camera -->
@@ -18,13 +17,14 @@
     <origin xyz="0.0675 0.2 0.54" rpy="0 -0 1.5707" />
   </xacro:camera_rc2016>
-  <!-- realsense d435
+  <!-- realsense d435 -->
   <xacro:include filename="$(find realsense_gazebo_plugin)/urdf/realsense_d435.urdf.xacro"/>
   <xacro:realsense_d435 parent="base_link">
-    <origin xyz="0.0 0 0.54" rpy="1.5707 0 1.5707" />
-  </xacro:realsense_d435> -->
-  <!-- realsense d455 -->
+    <origin xyz="-0.0905 -0.0905 1.73" rpy="1.9633 0 1.5707" />
+                                              <!-- rpy   v    0   h -->
+  </xacro:realsense_d435>
+  <!-- realsense d455
   <xacro:include filename="$(find realsense_gazebo_plugin)/urdf/realsense_d455.urdf.xacro"/>
   <xacro:realsense_d455 parent="base_link">
     <origin xyz="0.0 0 $(arg camera_height)" rpy="1.5707 0 1.5707" />
-  </xacro:realsense_d455>
+  </xacro:realsense_d455> -->
 </robot>
